File: pcb/keypad/keypad.kicad_pcb (KiCad board)
At the start: 2 copper layers, 208.3 x 86.4 mm, 49 parts, among them J1 Conn_02x05_Counter_Clockwise, M1 MountingHole_2.1mm, M2 MountingHole_2.1mm, M3 MountingHole_2.1mm, M4 MountingHole_2.1mm, SW1 SW_Push, SW10 SW_Push, SW11 SW_Push, SW12 SW_Push, SW13 SW_Push, SW14 SW_Push, SW15 SW_Push, SW16 SW_Push, SW17 SW_Push, SW18 SW_Push, SW19 SW_Push, SW2 SW_Push, SW20 SW_Push, SW21 SW_Push, SW22 SW_Push, SW23 SW_Push, SW24 SW_Push, SW25 SW_Push, SW26 SW_Push, SW27 SW_Push, SW28 SW_Push, SW29 SW_Push, SW3 SW_Push, SW30 SW_Push, SW31 SW_Push, SW32 SW_Push, SW33 SW_Push, SW34 SW_Push, SW35 SW_Push, SW36 SW_Push, SW4 SW_Push, SW5 SW_Push, SW6 SW_Push, SW7 SW_Push, SW8 SW_Push, SW9 SW_Push, U1 74HC595

Commit message: annotated pinout
Other:
- board text added: "5V"
- board text added: "clk"
- board text added: "gnd"
- board text added: "ld"
- board text added: "r1"
- board text added: "r2"
- board text added: "r3"
- board text added: "r4"
- board text added: "r5"
- board text added: "r6"
Changed lines of the file:
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@@
   (gr_line (start 22.86 25.4) (end 231.14 25.4) (layer "Edge.Cuts") (width 0.1))
   (gr_line (start 231.14 111.76) (end 22.86 111.76) (layer "Edge.Cuts") (width 0.1))
+  (gr_text "r6\n" (at 63.5 95.25 90) (layer "F.SilkS")
+    (effects (font (size 1.5 1.5) (thickness 0.3)))
+  )
+  (gr_text "r1\n\n" (at 69.85 85.09 90) (layer "F.SilkS")
+    (effects (font (size 1.5 1.5) (thickness 0.3)))
+  )
   (gr_text "Picochord Keypad\nGarnet Grimm 2022" (at 170.18 96.52) (layer "F.SilkS")
     (effects (font (size 1 1) (thickness 0.15)))
   )
+  (gr_text "ld\n\n" (at 72.39 85.09 90) (layer "F.SilkS")
+    (effects (font (size 1.5 1.5) (thickness 0.3)))
+  )
+  (gr_text "clk\n" (at 71.12 95.25 90) (layer "F.SilkS")
+    (effects (font (size 1.5 1.5) (thickness 0.3)))
+  )
+  (gr_text "r2\n" (at 66.04 85.09 90) (layer "F.SilkS")
+    (effects (font (size 1.5 1.5) (thickness 0.3)))
+  )
+  (gr_text "r4\n" (at 68.58 95.25 90) (layer "F.SilkS")
+    (effects (font (size 1.5 1.5) (thickness 0.3)))
+  )
+  (gr_text "r5\n" (at 66.04 95.25 90) (layer "F.SilkS")
+    (effects (font (size 1.5 1.5) (thickness 0.3)))
+  )
+  (gr_text "5V" (at 73.66 95.25 90) (layer "F.SilkS")
+    (effects (font (size 1.5 1.5) (thickness 0.3)))
+  )
+  (gr_text "r3\n" (at 63.5 85.09 90) (layer "F.SilkS")
+    (effects (font (size 1.5 1.5) (thickness 0.3)))
+  )
+  (gr_text "gnd\n" (at 73.66 83.82 90) (layer "F.SilkS")
+    (effects (font (size 1.5 1.5) (thickness 0.3)))
+  )
   (segment (start 116.86 96.52) (end 132.1 96.52) (width 0.25) (layer "B.Cu") (net 1))
