File: pcb/speaker/speaker.kicad_pcb (KiCad board)
At the start: 2 copper layers, 80 x 72.4 mm, 19 parts, among them J1 Conn_01x03_Female, J2 Conn_01x02_Female, U1 LM386

Commit message: annotated pinout
Other:
- board text added: "9V"
- board text added: "gnd"
- board text added: "in"
- board text added: "out"
Changed lines of the file:
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@@
   )
   (gr_rect (start 144.78 130.81) (end 64.77 58.42) (layer "Edge.Cuts") (width 0.05) (fill none))
+  (gr_text "9V\n" (at 87.63 80.01) (layer "F.SilkS")
+    (effects (font (size 1.5 1.5) (thickness 0.3)))
+  )
+  (gr_text "out" (at 140.97 76.2) (layer "F.SilkS")
+    (effects (font (size 1.5 1.5) (thickness 0.3)))
+  )
+  (gr_text "gnd\n" (at 87.63 77.47) (layer "F.SilkS")
+    (effects (font (size 1.5 1.5) (thickness 0.3)))
+  )
+  (gr_text "in" (at 87.63 74.93) (layer "F.SilkS")
+    (effects (font (size 1.5 1.5) (thickness 0.3)))
+  )
+  (gr_text "gnd\n" (at 140.97 73.66) (layer "F.SilkS")
+    (effects (font (size 1.5 1.5) (thickness 0.3)))
+  )
   (segment (start 123.19 85.09) (end 123.19 71.12) (width 0.25) (layer "F.Cu") (net 1))
   (segment (start 111.78 92.71) (end 111.77 92.72) (width 0.25) (layer "F.Cu") (net 2))
