File: pcb/strumpad/strumpad.kicad_pcb (KiCad board)
At the start: 2 copper layers, 74.9 x 107.9 mm, 23 parts, among them J1 Conn_01x05, U1 74HC165

Commit message: annotated pinout
Other:
- board text added: "5V"
- board text added: "clk"
- board text added: "gnd"
- board text added: "ld"
- board text added: "out"
Changed lines of the file:
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@@
   )
   (gr_rect (start 176.53 25.4) (end 101.6 133.35) (layer "Edge.Cuts") (width 0.05) (fill none))
+  (gr_text "gnd" (at 104.14 82.55) (layer "F.SilkS")
+    (effects (font (size 1.5 1.5) (thickness 0.3)))
+  )
+  (gr_text "5V" (at 104.14 85.09) (layer "F.SilkS")
+    (effects (font (size 1.5 1.5) (thickness 0.3)))
+  )
+  (gr_text "clk" (at 104.14 74.93) (layer "F.SilkS")
+    (effects (font (size 1.5 1.5) (thickness 0.3)))
+  )
+  (gr_text "out" (at 104.14 80.01) (layer "F.SilkS")
+    (effects (font (size 1.5 1.5) (thickness 0.3)))
+  )
+  (gr_text "ld" (at 104.14 77.47) (layer "F.SilkS")
+    (effects (font (size 1.5 1.5) (thickness 0.3)))
+  )
   (segment (start 160.02 35.56) (end 160.02 38.1) (width 0.25) (layer "F.Cu") (net 1))
   (segment (start 156.2 36.82) (end 151.14 36.82) (width 0.25) (layer "F.Cu") (net 1))

Commit message: strumpad update'
Parts:
- moved J1 36.7 mm to (116.8, 39.4)
- moved REF** 14.4 mm to (115.6, 119.4)
- moved R1 10.2 mm to (172.7, 92.7)
- moved R2 10.2 mm to (165.1, 92.7)
- moved R3 10.2 mm to (157.5, 92.7)
- moved R4 10.2 mm to (149.9, 92.7)
- moved R5 10.2 mm to (142.2, 92.7)
- moved R6 10.2 mm to (134.6, 92.7)
- moved R7 10.2 mm to (127.0, 92.7)
- moved R8 10.2 mm to (119.4, 92.7)
- moved D1 10.2 mm to (172.7, 102.9)
- moved D2 10.2 mm to (165.1, 102.9)
- moved D3 10.2 mm to (157.5, 102.9)
- moved D4 10.2 mm to (149.9, 102.9)
- moved D5 10.2 mm to (142.2, 102.9)
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Routing:
- net p8: track 83.9 -> 41.4 mm, vias 2 -> 0
- net p7: track 75.3 -> 34.2 mm, vias 2 -> 0
- net clk: track 209.7 -> 168.7 mm
- net p6: track 65.8 -> 27.0 mm, vias 2 -> 0
- net VCC: track 109.0 -> 70.8 mm
- net p5: track 60.0 -> 22.7 mm, vias 2 -> 0
- net p4: track 59.2 -> 21.9 mm, vias 2 -> 0
- net p3: track 62.5 -> 26.7 mm, vias 2 -> 0
- net p2: track 72.7 -> 36.8 mm, vias 2 -> 0
- net p1: track 82.1 -> 47.0 mm, vias 2 -> 0
- net ld: track 64.6 -> 29.8 mm
- net GND: track 95.6 -> 61.8 mm
- net out: track 62.3 -> 28.8 mm
Other:
- board size 74.9 x 107.9 mm -> 64.8 x 99.1 mm
